File: untitled-bruecke.brd (EAGLE design)
At the start: 122 x 86 mm, 16 parts, among them U1 C-TEENSY++

Commit message: Turn board and schematic into new revision: “kinX”
The new controller revision uses a Teensy 3.6, which requires some rewiring.

I used the chance to perform a bunch of cleanups:

• Use SMD LEDs instead of THT (resistors were already SMD)
• Move LED silkscreen labels to the correct side
• Correct the names of all connectors to match the kinesis PCBs
• Change the matrix to be easier to wire up
Parts:
- LED1, LED2, LED3, LED4: device led:LED3MM -> led:SML1206
- U1: value C-TEENSY++ -> TEENSY_3.5/3.6; device teensypp:TEENSY++ -> Teensy356:TEENSY_3.5/3.6
- moved U1 2.34 mm to (63.0, 46.2), flipped to the bottom, turned to 0 degrees
- moved LED1 0.50 mm to (45.8, 4.00), turned to 270 degrees
- moved LED2 0.50 mm to (56.0, 4.00), turned to 270 degrees
- moved LED3 0.50 mm to (66.0, 4.00), turned to 270 degrees
- moved LED4 0.50 mm to (76.2, 4.00), turned to 270 degrees
- renumbered DAUMENLINKS to THUMB_RIGHT_SPC, DAUMENRECHTS to THUMB_LEFT_BAK, TASTENLINKS to LEFT_13_LT, TASTENRECHTS to RGHT_13_DOWN, TOPLINKS to TOP_LEFT, TOPRECHTS to TOP_RIGHT
Connections:
- removed net B0: LEFT_13_LT.P$1, RGHT_13_DOWN.P$10, TOP_LEFT.P$1, U1.B0
- removed net B1: LEFT_13_LT.P$9, RGHT_13_DOWN.P$9, TOP_LEFT.P$8, U1.B1
- removed net B2: LEFT_13_LT.P$11, RGHT_13_DOWN.P$8, TOP_LEFT.P$5, U1.B2
- removed net B3: LEFT_13_LT.P$12, RGHT_13_DOWN.P$7, TOP_RIGHT.P$8, U1.B3
- removed net B4: LEFT_13_LT.P$13, RGHT_13_DOWN.P$4, TOP_RIGHT.P$5, U1.B4
- removed net B5: THUMB_LEFT_BAK.5, THUMB_RIGHT_SPC.8, TOP_RIGHT.P$10, TOP_RIGHT.P$11, U1.B5
- removed net B6: THUMB_LEFT_BAK.4, THUMB_RIGHT_SPC.7, U1.B6
- removed net C0: RGHT_13_DOWN.P$2, THUMB_RIGHT_SPC.5, U1.C0
- removed net C1: RGHT_13_DOWN.P$12, THUMB_RIGHT_SPC.6, U1.C1
- removed net C2: RGHT_13_DOWN.P$13, U1.C2
- removed net C3: RGHT_13_DOWN.P$6, U1.C3
- removed net C4: TOP_LEFT.P$2, TOP_RIGHT.P$9, U1.C4
- removed net C5: TOP_LEFT.P$10, TOP_LEFT.P$3, TOP_LEFT.P$6, TOP_RIGHT.P$13, TOP_RIGHT.P$3, TOP_RIGHT.P$6, U1.C5
- removed net C6: TOP_LEFT.P$11, TOP_LEFT.P$4, TOP_LEFT.P$7, TOP_RIGHT.P$12, TOP_RIGHT.P$4, TOP_RIGHT.P$7, U1.C6
- removed net D0: LEFT_13_LT.P$8, U1.D0
- removed net D1: LEFT_13_LT.P$7, U1.D1
- removed net D2: LEFT_13_LT.P$6, THUMB_LEFT_BAK.2, U1.D2
- removed net D3: LEFT_13_LT.P$4, THUMB_LEFT_BAK.8, U1.D3
- removed net D4: LEFT_13_LT.P$3, THUMB_LEFT_BAK.1, U1.D4
- removed net D5: LEFT_13_LT.P$2, THUMB_LEFT_BAK.3, U1.D5
- removed net D6: RGHT_13_DOWN.P$1, THUMB_RIGHT_SPC.3, U1.D6
- removed net D7: RGHT_13_DOWN.P$3, THUMB_RIGHT_SPC.4, U1.D7
- removed net N$1: U1.GND
- removed net N$11: LED1.A, LED2.A, LED3.A, LED4.A, U1.+5V
- new net 3V3: LED1.A, LED2.A, LED3.A, LED4.A, U1.3V3
- new net COL0: LEFT_13_LT.P$1, RGHT_13_DOWN.P$10, TOP_LEFT.P$8, U1.20/A6
- new net COL1: LEFT_13_LT.P$9, RGHT_13_DOWN.P$9, TOP_LEFT.P$5, U1.21/A7
- new net COL2: LEFT_13_LT.P$11, RGHT_13_DOWN.P$8, TOP_LEFT.P$1, U1.8
- new net COL3: LEFT_13_LT.P$12, RGHT_13_DOWN.P$7, TOP_RIGHT.P$8, U1.7
- new net COL4: LEFT_13_LT.P$13, RGHT_13_DOWN.P$4, TOP_RIGHT.P$5, U1.6
- new net COL5: THUMB_LEFT_BAK.5, THUMB_RIGHT_SPC.8, TOP_RIGHT.P$10, TOP_RIGHT.P$11, U1.14/A0
- new net COL6: THUMB_LEFT_BAK.4, THUMB_RIGHT_SPC.7, U1.2
- new net ROW_0: RGHT_13_DOWN.P$13, U1.5
- new net ROW_1: LEFT_13_LT.P$7, U1.28
- new net ROW_2: LEFT_13_LT.P$6, THUMB_LEFT_BAK.8, U1.29
- new net ROW_3: LEFT_13_LT.P$4, THUMB_LEFT_BAK.3, U1.30
- new net ROW_4: LEFT_13_LT.P$3, THUMB_LEFT_BAK.2, U1.31/A12
- new net ROW_5: LEFT_13_LT.P$2, THUMB_LEFT_BAK.1, U1.32/A13
- new net ROW_6: RGHT_13_DOWN.P$12, THUMB_RIGHT_SPC.3, U1.4/CANRX
- new net ROW_7: RGHT_13_DOWN.P$3, THUMB_RIGHT_SPC.4, U1.3/CANTX
- new net ROW_8: RGHT_13_DOWN.P$2, THUMB_RIGHT_SPC.5, U1.0/RX
- new net ROW_9: RGHT_13_DOWN.P$1, THUMB_RIGHT_SPC.6, U1.1/TX
- new net ROW_EQL: LEFT_13_LT.P$8, U1.27
- new net ROW_ESC: TOP_LEFT.P$2, TOP_RIGHT.P$9, U1.38/A19
- new net ROW_F1: TOP_LEFT.P$10, TOP_LEFT.P$3, TOP_LEFT.P$6, TOP_RIGHT.P$13, TOP_RIGHT.P$3, TOP_RIGHT.P$6, U1.37/A18
- new net ROW_F2: TOP_LEFT.P$11, TOP_LEFT.P$4, TOP_LEFT.P$7, TOP_RIGHT.P$12, TOP_RIGHT.P$4, TOP_RIGHT.P$7, U1.36/A17
- new net ROW_MIN: RGHT_13_DOWN.P$6, U1.9/CS
- net GND: now also U1.GND; no longer U1.GRND1
- net N$10: now also R1.2, U1.26; no longer R4.2, U1.F0
- net N$14: now also LED4.C; no longer LED4.K
- net N$15: now also LED3.C; no longer LED3.K
- net N$16: now also LED2.C; no longer LED2.K
- net N$17: now also LED1.C; no longer LED1.K
- net N$7: now also R4.2, U1.12/MISO; no longer R1.2, U1.F3
- net N$8: now also R3.2, U1.24; no longer R2.2, U1.F2
- net N$9: now also R2.2, U1.25; no longer R3.2, U1.F1
Routing:
- net COL5: track 0.00 -> 229.0 mm, vias 0 -> 2
- net COL1: track 0.00 -> 206.6 mm
- net COL2: track 0.00 -> 178.9 mm, vias 0 -> 1
- net COL4: track 0.00 -> 176.1 mm, vias 0 -> 1
- net COL0: track 0.00 -> 176.0 mm, vias 0 -> 1
- net B5: track 175.4 -> 0.00 mm, vias 1 -> 0
- net B4: track 172.5 -> 0.00 mm, vias 1 -> 0
- net COL3: track 0.00 -> 169.7 mm, vias 0 -> 1
- net B2: track 167.9 -> 0.00 mm, vias 1 -> 0
- net B3: track 166.9 -> 0.00 mm, vias 1 -> 0
- net B1: track 162.9 -> 0.00 mm, vias 1 -> 0
- net B0: track 150.9 -> 0.00 mm
- net D6: track 144.6 -> 0.00 mm
- net D7: track 143.6 -> 0.00 mm
- net ROW_F1: track 0.00 -> 140.6 mm, vias 0 -> 1
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Other:
- board text added: "CAPS_LOCK"
- board text added: "NUM_LOCK"
- board text added: "SCROLL_LOCK"
- board text added: "kinX keyboard controller"
- board text added: "v2017-12-09"
- board text removed: "18.03.2013"
- board text removed: "CAPS"
- board text removed: "NUM"
- board text removed: "SCR"
- board text removed: "Teensy++ Kinesis controller"
