File: kinx.brd (EAGLE design)
At the start: 122 x 86 mm, 16 parts, among them U1 TEENSY_3.5/3.6

Commit message: schematic: fix ROW_6/ROW_9 (they were swapped)
Connections:
- net ROW_6: now also RGHT_13_DOWN.P$1, THUMB_RIGHT_SPC.6, U1.1/TX; no longer RGHT_13_DOWN.P$12, THUMB_RIGHT_SPC.3, U1.4/CANRX
- net ROW_9: now also RGHT_13_DOWN.P$12, THUMB_RIGHT_SPC.3, U1.4/CANRX; no longer RGHT_13_DOWN.P$1, THUMB_RIGHT_SPC.6, U1.1/TX
Routing:
- net ROW_9: track 91.4 -> 62.2 mm, vias 0 -> 2
- net ROW_6: track 62.2 -> 91.4 mm, vias 2 -> 0
Changed lines of the file:
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@@
 <wire x1="115" y1="36" x2="89" y2="36" width="0.4064" layer="1"/>
 </signal>
-<signal name="ROW_9">
+<signal name="ROW_6">
 <contactref element="THUMB_RIGHT_SPC" pad="6"/>
 <wire x1="100.77" y1="10.27" x2="100.77" y2="7" width="0.4064" layer="1"/>
@@
 <wire x1="40.16" y1="34.16" x2="39" y2="33" width="0.4064" layer="16"/>
 </signal>
-<signal name="ROW_6">
+<signal name="ROW_9">
 <contactref element="THUMB_RIGHT_SPC" pad="3"/>
 <wire x1="101" y1="31" x2="101.75" y2="31.75" width="0.4064" layer="1"/>
