File: kint.kicad_pcb (KiCad board)
At the start: 2 copper layers, 122 x 86 mm, 23 parts, among them J1 THUMB_RIGHT_SPC_KB600, J2 LEFT_13_LT, J3 TOP_LEFT, J4 TOP_RIGHT, J5 THUMB_LEFT_BAK, J6 THUMB_RIGHT_SPC, J7 RIGHT_13_DOWN, J8 THUMB_LEFT_BAK_KB600, U1 TEENSY_3.5_3.6

Commit message: more silkscreen improvements
Parts:
- added G***: LOGO, kinx:logo, F.Cu at (122.4, 77.9)
- U1: value TEENSY_3.5_3.6 -> TEENSY_3.5/3.6
Other:
- board text added: "(L) = only caps lock LED"
